File: a-wai/Evil Head/Evil Head.sch (KiCad schematic (older format))
At the start: 84 parts, among them J1 JACK-MONOSW, K1 G5V2, P1 RLY+, P10 FROM PRE+, P11 Ug2, P12 Ubias, P13 FROM PRE-, P2 RLY-, P3 HT, P4 TO CLN EQ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

Commit message: Update Evil Head & add Evil Eddie
Parts:
- removed P4: TO CLN EQ, A-wai_Turrets:TURRET, symbol CONN_01X01
- removed P5: FROM CLN EQ, A-wai_Turrets:TURRET, symbol CONN_01X01
- removed P6: FROM LD EQ, A-wai_Turrets:TURRET, symbol CONN_01X01
- removed P7: TO LD EQ, A-wai_Turrets:TURRET, symbol CONN_01X01
- removed R35, R36: 10k, A-wai_Turrets:R_0.5W, symbol R
- added C?: 500p, A-wai_Turrets:C_225P_104_400V, symbol C
- added C? (x2): 22n, A-wai_Turrets:C_225P_104_400V, symbol C
- added C?: 250p, A-wai_Turrets:C_225P_104_400V, symbol C
- added C?: 100n, A-wai_Turrets:C_225P_104_400V, symbol C
- added C?: 47n, A-wai_Turrets:C_225P_104_400V, symbol C
- added C?: 22p, A-wai_Turrets:C_225P_104_400V, symbol C
- added R?: 22k, A-wai_Turrets:R_0.5W, symbol R
- added R?: 68k, A-wai_Turrets:R_0.5W, symbol R
- added R? (x3): 10k, A-wai_Turrets:R_0.5W, symbol R
- added RV? (x2): 250k-B, A-wai_Turrets:POT_13, symbol POT-RESCUE-Evil_Head
- added RV? (x3): 1M-A, A-wai_Turrets:POT_13, symbol POT-RESCUE-Evil_Head
- added RV?: 50k-B, A-wai_Turrets:POT_13, symbol POT-RESCUE-Evil_Head
- added RV?: 100k-B, A-wai_Turrets:POT_13, symbol POT-RESCUE-Evil_Head
- added RV?: 250k-A, A-wai_Turrets:POT_13, symbol POT-RESCUE-Evil_Head
- added RV?: 100k-A, A-wai_Turrets:POT_13, symbol POT-RESCUE-Evil_Head
- C16, C18: value 47n -> 100n
- RV1, RV2, RV3, RV4: symbol POT -> POT-RESCUE-Evil_Head
Connections:
- net GND: now also R?.2, RV?.3, RV?.3, RV?.3, RV?.3
- net HT_U3B: now also C?.1
- net at U1.2 (G): now also R?.1
- net at R14.2, R15.1: now also R?.2; no longer U2.2 (G)
- net at K1.11 (O), R11.1: now also C?.1, R?.2
- net at K1.8 (S): now also RV?.2
- net at RV3.1: now also C16.2
- net at RV4.1: now also C18.2
- new net: R?.1, U2.2 (G)
- new net: C?.2, RV?.1 (x2)
- new net: C?.1, C?.1, RV?.2, RV?.3
- new net: C?.2, RV?.1, RV?.2, RV?.3 (x2)
- new net: C?.2, RV?.2
- new net: RV?.1, RV?.2
- new net: RV?.1, RV?.3
- new net: R?.2, RV?.1
- new net: C?.1, C?.1, R?.1
- new net: C?.2, RV?.1, RV?.2
- new net: C?.1, RV?.1, RV?.2
- new net: R?.1, RV?.3
- new net: C?.2, R?.2, RV?.2
Other:
- moved on the sheet: C10, C11, C12, C9, D1, K1A, P1, P2, R11, R16, R17, R18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
