File: a-wai/Dirty Greed/Dirty Greed PCB.kicad_pcb (KiCad board)
At the start: 2 copper layers, 299.5 x 120 mm, 69 parts, among them J10 CRUNCH, J14 R+, J15 CR VOL, J16 LD VOL, J19 CR/LD, J21 PI GND, J26 BIAS, J27 EARTH, J7 CR GND, K2 FINDER-30.22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

Commit message: Dirty Greed: cut PCB some more
Parts:
- added REF**: MountingHole_3.5mm, MountingHole:MountingHole_3.5mm, F.Cu at (242.2, 70.2)
- moved REF** 45.3 mm to (319.8, 115.5)
Other:
- outline, holes or cut-outs redrawn
Changed lines of the file:
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@@
+	(footprint "MountingHole:MountingHole_3.5mm"
+		(layer "F.Cu")
+		(at 242.25 70.25)
+		(descr "Mounting Hole 3.5mm, no annular")
+		(tags "mounting hole 3.5mm no annular")
+		(property "Reference" "REF**"
+			(at 0 -4.5 0)
+			(layer "F.SilkS")
+			(hide yes)
+			(effects
+				(font
+					(size 1 1)
+					(thickness 0.15)
+				)
+			)
+		)
+		(property "Value" "MountingHole_3.5mm"
+			(at 0 4.5 0)
+			(layer "F.Fab")
+			(hide yes)
+			(effects
+				(font
+					(size 1 1)
+					(thickness 0.15)
+				)
+			)
+		)
+		(property "Datasheet" ""
+			(at 0 0 0)
+			(unlocked yes)
+			(layer "F.Fab")
+			(hide yes)
+			(effects
+				(font
+					(size 1.27 1.27)
+					(thickness 0.15)
+				)
+			)
+		)
+		(property "Description" ""
+			(at 0 0 0)
+			(unlocked yes)
+			(layer "F.Fab")
+			(hide yes)
+			(effects
+				(font
+					(size 1.27 1.27)
+					(thickness 0.15)
+				)
+			)
+		)
+		(clearance 2)
+		(attr exclude_from_pos_files exclude_from_bom)
+		(fp_circle
+			(center 0 0)
+			(end 3.5 0)
+			(stroke
+				(width 0.15)
+				(type solid)
+			)
+			(fill no)
+			(layer "Cmts.User")
+		)
+		(fp_circle
+			(center 0 0)
+			(end 3.75 0)
+			(stroke
+				(width 0.05)
+				(type solid)
+			)
+			(fill no)
+			(layer "F.CrtYd")
+		)
+		(pad "" np_thru_hole circle
+			(at 0 0)
+			(size 3.5 3.5)
+			(drill 3.5)
+			(layers "*.Cu" "*.Mask")
+		)
+		(embedded_fonts no)
+	)
 	(footprint "MountingHole:MountingHole_3.5mm"
 		(layer "F.Cu")
@@
 	(footprint "MountingHole:MountingHole_3.5mm"
 		(layer "F.Cu")
-		(at 319 70.25)
+		(at 319.75 115.5)
 		(descr "Mounting Hole 3.5mm, no annular")
 		(tags "mounting hole 3.5mm no annular")
@@
 	)
 	(gr_line
-		(start 324.5 68)
+		(start 324.5 113.5)
 		(end 324.5 182)
 		(stroke
@@
 	(gr_line
 		(start 28 65)
-		(end 321.5 65)
+		(end 244.302086 65.052086)
 		(stroke
 			(width 0.1)
@@
 	)
 	(gr_line
-		(start 324.5 68)
-		(end 321.5 65)
+		(start 289.697914 110.447914)
+		(end 244.302086 65.052086)
 		(stroke
 			(width 0.1)
@@
 		(stroke
 			(width 0.1)
+			(type solid)
+		)
+		(layer "Edge.Cuts")
+	)
+	(gr_line
+		(start 324.5 113.5)
+		(end 321.5 110.5)
+		(stroke
+			(width 0.1)
+			(type solid)
+		)
+		(layer "Edge.Cuts")
+	)
+	(gr_line
+		(start 289.697914 110.447914)
+		(end 321.48609 110.48609)
+		(stroke
+			(width 0.1)
